File: mphase.X/board/mphase.brd (EAGLE design)
At the start: 120.6 x 82.2 mm, 36 parts, among them IC1 MAX232, IC2 PIC18F4455_40, X1 332-10, X2 332-10

Commit message: up
Parts:
- added JP1: (no value), pinhead:1X07
- added R10, R11: 2.2k, resistor:0204V
- C1, C2, C3, C4: device resistor:C025-025X050 -> rcl:C1206
- moved C7 8.03 mm to (87.6, 41.9), turned to 90 degrees
- moved C1 7.62 mm to (101.6, 44.5)
- moved C4 6.35 mm to (95.2, 44.5)
- moved C2 1.27 mm to (101.6, 39.4), turned to 180 degrees
- moved C3 1.27 mm to (95.2, 39.4), turned to 180 degrees
Connections:
- new net N$37: IC2.21, JP1.2
- new net RD0: IC2.19, JP1.3, R11.2
- new net RD1: IC2.20, JP1.4, R10.1
- net N$5: now also C4.2; no longer C3.2
- net N$6: now also C3.1; no longer C4.1
- net VDD: now also R10.2, R11.1
- net VSS: now also C3.2, C4.1, JP1.6, JP1.7; no longer C3.1, C4.2
Routing:
- net N$11: track 171.5 -> 129.9 mm
- net RD0: track 0.00 -> 39.3 mm
- net N$12: track 166.3 -> 129.7 mm, vias 0 -> 1
- net N$10: track 119.6 -> 147.6 mm, vias 2 -> 1
- net VDD: track 199.4 -> 223.9 mm
- net N$37: track 0.00 -> 24.4 mm
- net N$26: track 51.6 -> 74.1 mm
- net RD1: track 0.00 -> 22.4 mm
- net N$32: track 30.6 -> 51.3 mm, vias 1 -> 0
- net N$17: track 67.6 -> 88.0 mm, vias 2 -> 0
- net N$31: track 47.4 -> 28.9 mm, vias 0 -> 1
- net N$13: track 134.9 -> 117.3 mm
- net N$23: track 53.5 -> 69.4 mm, vias 0 -> 1
- net N$33: track 65.9 -> 50.0 mm, vias 1 -> 0
- net N$16: track 81.1 -> 67.4 mm
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
Commit message: up
Parts:
- C10, C12, C8, C9: value 0.1 -> 0.1uf; device resistor:C025-024X044 -> rcl:C1206
- C11, C7: value 22uf -> 10uf; device resistor:C025-025X050 -> rcl:C1206
- C5: device resistor:C025-025X050 -> rcl:C1206
- C6: value 0.1 -> 0.1uf; device resistor:C025-025X050 -> rcl:C1206
- moved C7 65.9 mm to (27.9, 69.8), flipped to the bottom, turned to 0 degrees
- moved C8 57.1 mm to (81.3, 15.2), flipped to the bottom
- moved C10 36.0 mm to (35.6, 69.8), flipped to the bottom
- moved C5 34.9 mm to (43.2, 77.5), flipped to the bottom, turned to 180 degrees
- moved C6 26.7 mm to (41.9, 69.8), flipped to the bottom
- moved C9 17.8 mm to (36.8, 44.5), flipped to the bottom, turned to 180 degrees
- moved C12 7.73 mm to (29.2, 44.5), flipped to the bottom, turned to 180 degrees
- moved SV5 3.81 mm to (6.35, 39.4)
- moved C11 2.54 mm to (20.3, 22.9), flipped to the bottom
- flipped C1 to the bottom
- flipped C2 to the bottom
- flipped C3 to the bottom
- flipped C4 to the bottom
Connections:
- net N$37 renamed RD2
- removed net GND: C8.2, IC1.15, PL1.10, PL2.9, X1.9, X2.10
- removed net N$14: IC2.1, R3.2
- new net M_RST: C8.1, JP1.5, R1.2, R3.1
- net N$21: now also C10.2; no longer C9.1
- net N$22: now also C9.1; no longer C10.1
- net N$8: now also IC2.1, R3.2; no longer C8.1, R1.2, R3.1
- net VSS: now also C10.1, C8.2, IC1.15, PL1.10, PL2.9, X1.9, X2.10; no longer C10.2
Routing:
- net M_RST: track 0.00 -> 132.6 mm, vias 0 -> 1
- net GND: track 119.3 -> 0.00 mm
- net N$11: track 129.9 -> 175.6 mm, vias 0 -> 1
- net N$14: track 45.4 -> 0.00 mm
- net N$33: track 50.0 -> 81.9 mm, vias 0 -> 1
- net N$10: track 147.6 -> 116.4 mm, vias 1 -> 0
- net N$21: track 29.0 -> 54.6 mm, vias 1 -> 0
- net VCC: track 129.0 -> 107.3 mm
- net N$32: track 51.3 -> 30.6 mm
- net N$16: track 67.4 -> 87.9 mm
- net N$17: track 88.0 -> 74.7 mm
- net VSS: track 11.6 -> 0.00 mm
- net N$27: track 52.4 -> 60.7 mm, vias 1 -> 0
- net N$13: track 117.3 -> 109.2 mm, vias 1 -> 0
- net N$29: track 38.2 -> 30.5 mm
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